File: design_files/AST1012.brd (EAGLE design)
At the start: 10 x 10 mm, 7 parts, among them J1 SM05B, U1 TSL2572

Commit message: name change
Parts:
- C1: value 10uF -> 1uF
- J1: device tinycircuits:JST_SH_5X1 -> tinycircuits:JST_SH_5X1_EDGE
- R2: value 0.0 -> 1.00K
Other:
- board text added: "Wireling Light Sensor"
- board text removed: "Light Sensor Board"
Changed lines of the file:
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@@
 <layer number="59" name="Invisible" color="7" fill="1" visible="no" active="no"/>
 <layer number="61" name="stand" color="7" fill="1" visible="no" active="no"/>
+<layer number="88" name="SimResults" color="9" fill="1" visible="yes" active="yes"/>
+<layer number="89" name="SimProbes" color="9" fill="1" visible="yes" active="yes"/>
 <layer number="90" name="Modules" color="5" fill="1" visible="yes" active="yes"/>
 <layer number="91" name="Nets" color="2" fill="1" visible="no" active="no"/>
@@
 <layer number="158" name="bResistor" color="7" fill="1" visible="no" active="yes"/>
 <layer number="159" name="henwayCAP" color="13" fill="1" visible="yes" active="yes"/>
+<layer number="160" name="IDFDebug" color="7" fill="1" visible="yes" active="yes"/>
 <layer number="191" name="mNets" color="7" fill="1" visible="no" active="no"/>
 <layer number="192" name="mBusses" color="7" fill="1" visible="no" active="no"/>
@@
 <wire x1="0" y1="40.8" x2="0" y2="0" width="0.127" layer="48"/>
 <dimension x1="15" y1="20" x2="25" y2="20" x3="20" y3="21.454653125" layer="48"/>
-<text x="38.111025" y="4.365003125" size="0.889" layer="48">Light Sensor Board</text>
+<text x="38.111025" y="4.365003125" size="0.889" layer="48">Wireling Light Sensor</text>
 <text x="34.986825" y="1.7714" size="0.889" layer="48">AS-PCB-AST1012</text>
 <text x="57.3810375" y="1.6952" size="0.889" layer="48">2</text>
@@
 <attribute name="DATABASE" value="./../../../../../Components/TinyCircuits_Part_Database.txt" x="24.35" y="13.25" size="1.778" layer="27" rot="R90" display="off"/>
 </element>
-<element name="C1" library="tinycircuits" package="C0603" value="10uF" x="15.8" y="13.5" rot="R90">
-<attribute name="PARTNO" value="AS-ITM-00002" x="15.8" y="13.5" size="1.778" layer="27" rot="R90" display="off"/>
-<attribute name="VALUE" value="10uF" x="15.8" y="13.5" size="1.778" layer="27" rot="R90" display="off"/>
+<element name="C1" library="tinycircuits" package="C0603" value="1uF" x="15.8" y="13.5" rot="R90">
+<attribute name="PARTNO" value="AS-ITM-00410" x="15.8" y="13.5" size="1.778" layer="27" rot="R90" display="off"/>
+<attribute name="VALUE" value="1uF" x="15.8" y="13.5" size="1.778" layer="27" rot="R90" display="off"/>
 </element>
-<element name="J1" library="tinycircuits" package="JST_SH_5X1" value="SM05B" x="20" y="12.125">
+<element name="J1" library="tinycircuits" package="JST_SH_5X1_EDGE" value="SM05B" x="20" y="12.125">
 <attribute name="PARTNO" value="AS-ITM-00340" x="20" y="12.125" size="1.778" layer="27" display="off"/>
 <attribute name="VALUE" value="SM05B" x="20" y="12.125" size="1.778" layer="27" display="off"/>
+<attribute name="PNPROTATION" value="180" x="20" y="12.125" size="1.778" layer="27" display="off"/>
 </element>
-<element name="R2" library="tinycircuits" package="0402" value="0.0" x="23.7" y="14.9" rot="R180">
-<attribute name="PARTNO" value="AS-ITM-00076" x="23.7" y="14.9" size="1.778" layer="27" rot="R180" display="off"/>
-<attribute name="VALUE" value="0.0" x="23.7" y="14.9" size="1.778" layer="27" rot="R180" display="off"/>
+<element name="R2" library="tinycircuits" package="0402" value="1.00K" x="23.7" y="14.9" rot="R180">
+<attribute name="PARTNO" value="AS-ITM-00003" x="23.7" y="14.9" size="1.778" layer="27" rot="R180" display="off"/>
+<attribute name="VALUE" value="1.00K" x="23.7" y="14.9" size="1.778" layer="27" rot="R180" display="off"/>
 </element>
 <element name="U1" library="tinycircuits" package="TSL2572" value="TSL2572" x="20" y="18">
