File: design_files/AST1012.sch (EAGLE design)
At the start: 6 parts, among them J1 SM05B, U1 TSL2572

Commit message: name change
Parts:
- C1: value 10uF -> 1uF; device tinycircuits:AS-ITM-00002 -> tinycircuits:AS-ITM-00410; PARTNO (none) -> AS-ITM-00410; VALUE (none) -> 1uF
- J1: device tinycircuits:AS-ITM-00340 -> tinycircuits:AS-ITM-00340EDGE
- R2: value 0.0 -> 1.00K; device tinycircuits:AS-ITM-00076 -> tinycircuits:AS-ITM-00003; PARTNO (none) -> AS-ITM-00003; VALUE (none) -> 1.00K
Other:
- note added: "Variant: Standard - R"
- note added: "Wireling Light Sensor"
- note removed: "Light Sensor Board"
- note removed: "Variant: Standard"
